File: _autosave-Cognac Carl TKL+Macro Column Duplexed.sch (KiCad schematic (older format))
At the start: 277 parts

Commit message: Added Type-C connector, footprints
Parts:
- removed C?: 1uF, symbol Device:C_Small
- removed D? (x36): SOD-123, symbol Device:D
- removed MX_? (x10), MX_BSLS?, MX_BSPC?, MX_DEL?, MX_E?, MX_END?, MX_EQL?, MX_F? (x2), MX_GRAVE?, MX_HOME?, MX_I?, MX_INS?, MX_LBRC?, MX_MINS?, MX_O?, MX_P?, MX_PGDN?, MX_PGUP?, MX_Q?, MX_R?, MX_RBRC?, MX_T?, MX_TAB?, MX_U?, MX_W?, MX_Y?: MX-NoLED, symbol MX_Alps_Hybrid:MX-NoLED
- removed R?: 10k, symbol Device:R_Small
- removed R? (x2): 22, symbol Device:R_Small
- removed U?: AT90USB1286-MU, Package_DFN_QFN:QFN-64-1EP_9x9mm_P0.5mm_EP7.5x7.5mm, symbol MCU_Microchip_AVR:AT90USB1286-MU
Connections:
- net COL10 is gone; now on net COL5: MX_9.1 (COL), MX_DOT.1 (COL), MX_F8.1 (COL), MX_L.1 (COL), MX_O.1 (COL)
- net COL11 is gone; now on net COL5: MX_0.1 (COL), MX_F9.1 (COL), MX_P.1 (COL), MX_RALT.1 (COL), MX_SCLN.1 (COL), MX_SLSH.1 (COL)
- net COL12 is gone; now on net COL6: MX_F10.1 (COL), MX_LBRC.1 (COL), MX_MINS.1 (COL), MX_QUOT.1 (COL), MX_RWIN.1 (COL)
- net COL13 is gone; now on net COL6: MX_EQL.1 (COL), MX_F11.1 (COL), MX_MENU.1 (COL), MX_RBRC.1 (COL)
- net COL14 is gone; now on net COL7: MX_BSLS.1 (COL), MX_BSPC.1 (COL), MX_ENT.1 (COL), MX_F12.1 (COL), MX_RCTL.1 (COL), MX_RSFT.1 (COL)
- net COL15 is gone; now on net COL7: MX_DEL.1 (COL), MX_INS.1 (COL), MX_LEFT.1 (COL), MX_PSCR.1 (COL)
- net COL16 is gone; now on net COL8: MX_DOWN.1 (COL), MX_END.1 (COL), MX_HOME.1 (COL), MX_SLCK.1 (COL), MX_UP.1 (COL)
- net COL17 is gone; now on net COL8: MX_PAUS.1 (COL), MX_PGDN.1 (COL), MX_PGUP.1 (COL), MX_RGHT.1 (COL)
- net COL9 is gone; now on net COL4: MX_8.1 (COL), MX_COMM.1 (COL), MX_F7.1 (COL), MX_I.1 (COL), MX_K.1 (COL)
- net COL0: now also MX_CAPS.1 (COL), MX_ESC.1 (COL), MX_GRAVE.1 (COL), MX_LCTL.1 (COL), MX_LSFT.1 (COL), MX_TAB.1 (COL)
- net COL1: now also MX_1.1 (COL), MX_2.1 (COL), MX_A.1 (COL), MX_F1.1 (COL), MX_LALT.1 (COL), MX_LWIN.1 (COL), MX_Q.1 (COL), MX_S.1 (COL), MX_W.1 (COL), MX_X.1 (COL), MX_Z.1 (COL); no longer MX_CAPS.1 (COL), MX_ESC.1 (COL), MX_GRAVE.1 (COL), MX_LCTL.1 (COL), MX_LSFT.1 (COL), MX_TAB.1 (COL)
- net COL2: now also MX_3.1 (COL), MX_4.1 (COL), MX_C.1 (COL), MX_D.1 (COL), MX_E.1 (COL), MX_F.1 (COL), MX_F2.1 (COL), MX_F3.1 (COL), MX_R.1 (COL), MX_V.1 (COL); no longer MX_1.1 (COL), MX_A.1 (COL), MX_LWIN.1 (COL), MX_Q.1 (COL), MX_Z.1 (COL)
- net COL3: now also MX_5.1 (COL), MX_6.1 (COL), MX_B.1 (COL), MX_F4.1 (COL), MX_F5.1 (COL), MX_G.1 (COL), MX_H.1 (COL), MX_N.1 (COL), MX_SPC.1 (COL), MX_T.1 (COL), MX_Y.1 (COL); no longer MX_2.1 (COL), MX_F1.1 (COL), MX_LALT.1 (COL), MX_S.1 (COL), MX_W.1 (COL), MX_X.1 (COL)
- net COL4: now also MX_7.1 (COL), MX_F6.1 (COL), MX_J.1 (COL), MX_M.1 (COL), MX_U.1 (COL); no longer MX_3.1 (COL), MX_C.1 (COL), MX_D.1 (COL), MX_E.1 (COL), MX_F2.1 (COL)
- net COL5: no longer MX_4.1 (COL), MX_F.1 (COL), MX_F3.1 (COL), MX_R.1 (COL), MX_V.1 (COL)
- net COL6: no longer MX_5.1 (COL), MX_B.1 (COL), MX_F4.1 (COL), MX_G.1 (COL), MX_T.1 (COL)
- net COL7: no longer MX_6.1 (COL), MX_F5.1 (COL), MX_H.1 (COL), MX_N.1 (COL), MX_SPC.1 (COL), MX_Y.1 (COL)
- net COL8: no longer MX_7.1 (COL), MX_F6.1 (COL), MX_J.1 (COL), MX_M.1 (COL), MX_U.1 (COL)
- net ROW0: no longer D?.1 (K), D?.1 (K), D?.1 (K), D?.1 (K), D?.1 (K), D?.1 (K), D?.1 (K), D?.1 (K), D?.1 (K)
- net ROW1: now also D?.1 (K), D?.1 (K), D?.1 (K), D?.1 (K), D?.1 (K), D?.1 (K), D?.1 (K), D?.1 (K), D?.1 (K); no longer D?.1 (K), D?.1 (K), D?.1 (K), D?.1 (K), D?.1 (K), D?.1 (K), D?.1 (K), D?.1 (K), D?.1 (K), D?.1 (K), D?.1 (K), D?.1 (K), D?.1 (K), D?.1 (K), D?.1 (K), D?.1 (K), D?.1 (K), D?.1 (K)
- net ROW2: now also D?.1 (K), D?.1 (K), D?.1 (K), D?.1 (K), D?.1 (K), D?.1 (K), D?.1 (K), D?.1 (K), D?.1 (K); no longer D?.1 (K), D?.1 (K), D?.1 (K), D?.1 (K), D?.1 (K), D?.1 (K), D?.1 (K), D?.1 (K), D?.1 (K), D?.1 (K), D?.1 (K), D?.1 (K), D?.1 (K), D?.1 (K), D?.1 (K), D?.1 (K), D?.1 (K), D?.1 (K)
- net ROW3: now also D?.1 (K), D?.1 (K), D?.1 (K), D?.1 (K), D?.1 (K), D?.1 (K), D?.1 (K), D?.1 (K), D?.1 (K); no longer D?.1 (K), D?.1 (K), D?.1 (K), D?.1 (K), D?.1 (K), D?.1 (K), D?.1 (K), D?.1 (K), D?.1 (K), D?.1 (K), D?.1 (K), D?.1 (K), D?.1 (K), D?.1 (K)
- net ROW4: now also D?.1 (K), D?.1 (K), D?.1 (K), D?.1 (K), D?.1 (K), D?.1 (K), D?.1 (K), D?.1 (K), D?.1 (K); no longer D?.1 (K), D?.1 (K), D?.1 (K), D?.1 (K), D?.1 (K), D?.1 (K), D?.1 (K), D?.1 (K), D?.1 (K), D?.1 (K), D?.1 (K), D?.1 (K), D?.1 (K), D?.1 (K)
- net ROW5: now also D?.1 (K), D?.1 (K), D?.1 (K), D?.1 (K), D?.1 (K), D?.1 (K), D?.1 (K), D?.1 (K), D?.1 (K); no longer D?.1 (K), D?.1 (K), D?.1 (K), D?.1 (K), D?.1 (K), D?.1 (K), D?.1 (K), D?.1 (K), D?.1 (K), D?.1 (K), D?.1 (K), D?.1 (K)
- new net ROW10: D?.1 (K), D?.1 (K), D?.1 (K), D?.1 (K), D?.1 (K), D?.1 (K)
- new net ROW11: D?.1 (K), D?.1 (K), D?.1 (K), D?.1 (K), D?.1 (K), D?.1 (K)
- new net ROW6: D?.1 (K), D?.1 (K), D?.1 (K), D?.1 (K), D?.1 (K), D?.1 (K), D?.1 (K)
- new net ROW7: D?.1 (K), D?.1 (K), D?.1 (K), D?.1 (K), D?.1 (K), D?.1 (K), D?.1 (K)
- new net ROW8: D?.1 (K), D?.1 (K), D?.1 (K), D?.1 (K), D?.1 (K), D?.1 (K), D?.1 (K)
- new net ROW9: D?.1 (K), D?.1 (K), D?.1 (K), D?.1 (K), D?.1 (K), D?.1 (K), D?.1 (K)
Other:
- moved on the sheet: C?, R?, SW?, U?, Y?
