File: Cognac Carl TKL+Macro Column Duplexed_01.sch (KiCad schematic (older format))
At the start: 277 parts

Commit message: Added Type-C connector, footprints
Parts:
- removed C?: 1uF, symbol Device:C_Small
- removed D? (x36): SOD-123, symbol Device:D
- removed F?: 500mA, symbol Device:Fuse
- removed MX_? (x10), MX_BSLS?, MX_BSPC?, MX_DEL?, MX_E?, MX_END?, MX_EQL?, MX_F? (x2), MX_GRAVE?, MX_HOME?, MX_I?, MX_INS?, MX_LBRC?, MX_MINS?, MX_O?, MX_P?, MX_PGDN?, MX_PGUP?, MX_Q?, MX_R?, MX_RBRC?, MX_T?, MX_TAB?, MX_U?, MX_W?, MX_Y?: MX-NoLED, symbol MX_Alps_Hybrid:MX-NoLED
- removed R?: 10k, symbol Device:R_Small
- removed R? (x2): 22, symbol Device:R_Small
- removed U?: AT90USB1286-MU, Package_DFN_QFN:QFN-64-1EP_9x9mm_P0.5mm_EP7.5x7.5mm, symbol MCU_Microchip_AVR:AT90USB1286-MU
- removed USB?: Molex-0548190589, symbol random-keyboard-parts:Molex-0548190589
- added F?: 500mA, symbol Device:Polyfuse_Small
- added R? (x2): 5.1k, symbol Device:R_Small
- added USB?: HRO-TYPE-C-31-M-12, symbol Type-C:HRO-TYPE-C-31-M-12
Connections:
- net COL10 is gone; now on net COL5: MX_9.1 (COL), MX_DOT.1 (COL), MX_F8.1 (COL), MX_L.1 (COL), MX_O.1 (COL)
- net COL11 is gone; now on net COL5: MX_0.1 (COL), MX_F9.1 (COL), MX_P.1 (COL), MX_RALT.1 (COL), MX_SCLN.1 (COL), MX_SLSH.1 (COL)
- net COL12 is gone; now on net COL6: MX_F10.1 (COL), MX_LBRC.1 (COL), MX_MINS.1 (COL), MX_QUOT.1 (COL), MX_RWIN.1 (COL)
- net COL13 is gone; now on net COL6: MX_EQL.1 (COL), MX_F11.1 (COL), MX_MENU.1 (COL), MX_RBRC.1 (COL)
- net COL14 is gone; now on net COL7: MX_BSLS.1 (COL), MX_BSPC.1 (COL), MX_ENT.1 (COL), MX_F12.1 (COL), MX_RCTL.1 (COL), MX_RSFT.1 (COL)
- net COL15 is gone; now on net COL7: MX_DEL.1 (COL), MX_INS.1 (COL), MX_LEFT.1 (COL), MX_PSCR.1 (COL)
- net COL16 is gone; now on net COL8: MX_DOWN.1 (COL), MX_END.1 (COL), MX_HOME.1 (COL), MX_SLCK.1 (COL), MX_UP.1 (COL)
- net COL17 is gone; now on net COL8: MX_PAUS.1 (COL), MX_PGDN.1 (COL), MX_PGUP.1 (COL), MX_RGHT.1 (COL)
- net COL9 is gone; now on net COL4: MX_8.1 (COL), MX_COMM.1 (COL), MX_F7.1 (COL), MX_I.1 (COL), MX_K.1 (COL)
- net +5V: now also F?.1
- net COL0: now also MX_CAPS.1 (COL), MX_ESC.1 (COL), MX_GRAVE.1 (COL), MX_LCTL.1 (COL), MX_LSFT.1 (COL), MX_TAB.1 (COL)
- net COL1: now also MX_1.1 (COL), MX_2.1 (COL), MX_A.1 (COL), MX_F1.1 (COL), MX_LALT.1 (COL), MX_LWIN.1 (COL), MX_Q.1 (COL), MX_S.1 (COL), MX_W.1 (COL), MX_X.1 (COL), MX_Z.1 (COL); no longer MX_CAPS.1 (COL), MX_ESC.1 (COL), MX_GRAVE.1 (COL), MX_LCTL.1 (COL), MX_LSFT.1 (COL), MX_TAB.1 (COL)
- net COL2: now also MX_3.1 (COL), MX_4.1 (COL), MX_C.1 (COL), MX_D.1 (COL), MX_E.1 (COL), MX_F.1 (COL), MX_F2.1 (COL), MX_F3.1 (COL), MX_R.1 (COL), MX_V.1 (COL); no longer MX_1.1 (COL), MX_A.1 (COL), MX_LWIN.1 (COL), MX_Q.1 (COL), MX_Z.1 (COL)
- net COL3: now also MX_5.1 (COL), MX_6.1 (COL), MX_B.1 (COL), MX_F4.1 (COL), MX_F5.1 (COL), MX_G.1 (COL), MX_H.1 (COL), MX_N.1 (COL), MX_SPC.1 (COL), MX_T.1 (COL), MX_Y.1 (COL); no longer MX_2.1 (COL), MX_F1.1 (COL), MX_LALT.1 (COL), MX_S.1 (COL), MX_W.1 (COL), MX_X.1 (COL)
- net COL4: now also MX_7.1 (COL), MX_F6.1 (COL), MX_J.1 (COL), MX_M.1 (COL), MX_U.1 (COL); no longer MX_3.1 (COL), MX_C.1 (COL), MX_D.1 (COL), MX_E.1 (COL), MX_F2.1 (COL)
- net COL5: no longer MX_4.1 (COL), MX_F.1 (COL), MX_F3.1 (COL), MX_R.1 (COL), MX_V.1 (COL)
- net COL6: no longer MX_5.1 (COL), MX_B.1 (COL), MX_F4.1 (COL), MX_G.1 (COL), MX_T.1 (COL)
- net COL7: no longer MX_6.1 (COL), MX_F5.1 (COL), MX_H.1 (COL), MX_N.1 (COL), MX_SPC.1 (COL), MX_Y.1 (COL)
- net COL8: no longer MX_7.1 (COL), MX_F6.1 (COL), MX_J.1 (COL), MX_M.1 (COL), MX_U.1 (COL)
- net D+: now also USB?.6 (DP1), USB?.8 (DP2)
- net D-: now also USB?.5 (DN2), USB?.7 (DN1)
- net GND: now also R?.1, R?.1, USB?.1 (GND), USB?.12 (GND), USB?.13 (SHIELD)
- net ROW0: no longer D?.1 (K), D?.1 (K), D?.1 (K), D?.1 (K), D?.1 (K), D?.1 (K), D?.1 (K), D?.1 (K), D?.1 (K)
- net ROW1: now also D?.1 (K), D?.1 (K), D?.1 (K), D?.1 (K), D?.1 (K), D?.1 (K), D?.1 (K), D?.1 (K), D?.1 (K); no longer D?.1 (K), D?.1 (K), D?.1 (K), D?.1 (K), D?.1 (K), D?.1 (K), D?.1 (K), D?.1 (K), D?.1 (K), D?.1 (K), D?.1 (K), D?.1 (K), D?.1 (K), D?.1 (K), D?.1 (K), D?.1 (K), D?.1 (K), D?.1 (K)
- net ROW2: now also D?.1 (K), D?.1 (K), D?.1 (K), D?.1 (K), D?.1 (K), D?.1 (K), D?.1 (K), D?.1 (K), D?.1 (K); no longer D?.1 (K), D?.1 (K), D?.1 (K), D?.1 (K), D?.1 (K), D?.1 (K), D?.1 (K), D?.1 (K), D?.1 (K), D?.1 (K), D?.1 (K), D?.1 (K), D?.1 (K), D?.1 (K), D?.1 (K), D?.1 (K), D?.1 (K), D?.1 (K)
- net ROW3: now also D?.1 (K), D?.1 (K), D?.1 (K), D?.1 (K), D?.1 (K), D?.1 (K), D?.1 (K), D?.1 (K), D?.1 (K); no longer D?.1 (K), D?.1 (K), D?.1 (K), D?.1 (K), D?.1 (K), D?.1 (K), D?.1 (K), D?.1 (K), D?.1 (K), D?.1 (K), D?.1 (K), D?.1 (K), D?.1 (K), D?.1 (K)
- net ROW4: now also D?.1 (K), D?.1 (K), D?.1 (K), D?.1 (K), D?.1 (K), D?.1 (K), D?.1 (K), D?.1 (K), D?.1 (K); no longer D?.1 (K), D?.1 (K), D?.1 (K), D?.1 (K), D?.1 (K), D?.1 (K), D?.1 (K), D?.1 (K), D?.1 (K), D?.1 (K), D?.1 (K), D?.1 (K), D?.1 (K), D?.1 (K)
- net ROW5: now also D?.1 (K), D?.1 (K), D?.1 (K), D?.1 (K), D?.1 (K), D?.1 (K), D?.1 (K), D?.1 (K), D?.1 (K); no longer D?.1 (K), D?.1 (K), D?.1 (K), D?.1 (K), D?.1 (K), D?.1 (K), D?.1 (K), D?.1 (K), D?.1 (K), D?.1 (K), D?.1 (K), D?.1 (K)
- net VCC: now also F?.2, USB?.11 (VBUS), USB?.2 (VBUS)
- new net: R?.2, USB?.10 (CC2)
- new net: R?.2, USB?.4 (CC1)
- new net ROW10: D?.1 (K), D?.1 (K), D?.1 (K), D?.1 (K), D?.1 (K), D?.1 (K)
- new net ROW11: D?.1 (K), D?.1 (K), D?.1 (K), D?.1 (K), D?.1 (K), D?.1 (K)
- new net ROW6: D?.1 (K), D?.1 (K), D?.1 (K), D?.1 (K), D?.1 (K), D?.1 (K), D?.1 (K)
- new net ROW7: D?.1 (K), D?.1 (K), D?.1 (K), D?.1 (K), D?.1 (K), D?.1 (K), D?.1 (K)
- new net ROW8: D?.1 (K), D?.1 (K), D?.1 (K), D?.1 (K), D?.1 (K), D?.1 (K), D?.1 (K)
- new net ROW9: D?.1 (K), D?.1 (K), D?.1 (K), D?.1 (K), D?.1 (K), D?.1 (K), D?.1 (K)
- no-connect marks 0 -> 2
Other:
- moved on the sheet: C?, R?, SW?, U?, Y?

Commit message: actually added usbc and footprints
Parts:
- C1, C2, C3, C4, C5, C6, C7: renamed from C?; footprint (none) -> Capacitor_SMD:C_0805_2012Metric
- D1, D10, D11, D12, D13, D14, D15, D16, D17, D18, D19, D2, D20, D21, D22, D23, D24, D25, D26, D27, D28, D29, D3, D30, D31, D32, D33, D34, D35, D36, D37, D38, D39, D4, D40, D41, D42, D43, D44, D45, D46, D47, D48, D49, D5, D50, D51, D52, D53, D54, D55, D56, D57, D58, D59, D6, D60, D61, D62, D63, D64, D65, D66, D67, D68, D69, D7, D70, D71, D72, D73, D74, D75, D76, D77, D78, D79, D8, D80, D81, D82, D83, D84, D85, D86, D87, D88, D89, D9, D90, D91, D92: renamed from D?; footprint (none) -> Diode_SMD:D_SOD-123
- F1: renamed from F?; footprint (none) -> Fuse:Fuse_1206_3216Metric
- MX_0, MX_1, MX_2, MX_3, MX_4, MX_5, MX_6, MX_7, MX_8, MX_9, MX_F1, MX_F10, MX_F11, MX_F12, MX_F13, MX_F14, MX_F15, MX_F16, MX_F17, MX_F2, MX_F3, MX_F4, MX_F5, MX_F6, MX_F7, MX_F8, MX_F9: footprint (none) -> MX_Only:MXOnly-1U-Hotswap
- MX_A1: renamed from MX_A; footprint (none) -> MX_Only:MXOnly-1U-Hotswap
- MX_B1: renamed from MX_B; footprint (none) -> MX_Only:MXOnly-1U-Hotswap
- MX_BSLS1: renamed from MX_BSLS; footprint (none) -> MX_Only:MXOnly-1.5U-Hotswap
- MX_BSPC1: renamed from MX_BSPC; footprint (none) -> MX_Only:MXOnly-2U-Hotswap
- MX_C1: renamed from MX_C; footprint (none) -> MX_Only:MXOnly-1U-Hotswap
- MX_CAPS1: renamed from MX_CAPS; value MX-NoLED -> MXOnly-1.75U-Hotswap; footprint (none) -> MX_Only:MXOnly-1.75U-Hotswap
- MX_COMM1: renamed from MX_COMM; footprint (none) -> MX_Only:MXOnly-1U-Hotswap
- MX_D1: renamed from MX_D; footprint (none) -> MX_Only:MXOnly-1U-Hotswap
- MX_DEL1: renamed from MX_DEL; footprint (none) -> MX_Only:MXOnly-1U-Hotswap
- MX_DOT1: renamed from MX_DOT; footprint (none) -> MX_Only:MXOnly-1U-Hotswap
- MX_DOWN1: renamed from MX_DOWN; footprint (none) -> MX_Only:MXOnly-1U-Hotswap
- MX_E1: renamed from MX_E; footprint (none) -> MX_Only:MXOnly-1U-Hotswap
- MX_END1: renamed from MX_END; footprint (none) -> MX_Only:MXOnly-1U-Hotswap
- MX_ENT1: renamed from MX_ENT; footprint (none) -> MX_Only:MXOnly-2.25U-Hotswap
- MX_EQL1: renamed from MX_EQL; footprint (none) -> MX_Only:MXOnly-1U-Hotswap
- MX_ESC1: renamed from MX_ESC; footprint (none) -> MX_Only:MXOnly-1U-Hotswap
- MX_F18: renamed from MX_F; footprint (none) -> MX_Only:MXOnly-1U-Hotswap
- MX_G1: renamed from MX_G; footprint (none) -> MX_Only:MXOnly-1U-Hotswap
- MX_GRAVE1: renamed from MX_GRAVE; footprint (none) -> MX_Only:MXOnly-1U-Hotswap
- MX_H1: renamed from MX_H; footprint (none) -> MX_Only:MXOnly-1U-Hotswap
- MX_HOME1: renamed from MX_HOME; footprint (none) -> MX_Only:MXOnly-1U-Hotswap
- MX_I1: renamed from MX_I; footprint (none) -> MX_Only:MXOnly-1U-Hotswap
- MX_INS1: renamed from MX_INS; footprint (none) -> MX_Only:MXOnly-1U-Hotswap
- MX_J1: renamed from MX_J; footprint (none) -> MX_Only:MXOnly-1U-Hotswap
- MX_K1: renamed from MX_K; footprint (none) -> MX_Only:MXOnly-1U-Hotswap
- MX_L1: renamed from MX_L; footprint (none) -> MX_Only:MXOnly-1U-Hotswap
- MX_LALT1: renamed from MX_LALT; value MX-NoLED -> MXOnly-1.25U-Hotswap; footprint (none) -> MX_Only:MXOnly-1.25U-Hotswap
- MX_LBRC1: renamed from MX_LBRC; footprint (none) -> MX_Only:MXOnly-1U-Hotswap
- MX_LCTL1: renamed from MX_LCTL; value MX-NoLED -> MXOnly-1.25U-Hotswap; footprint (none) -> MX_Only:MXOnly-1.25U-Hotswap
- MX_LEFT1: renamed from MX_LEFT; footprint (none) -> MX_Only:MXOnly-1U-Hotswap
- MX_LSFT1: renamed from MX_LSFT; value MX-NoLED -> MXOnly-2.25U-Hotswap; footprint (none) -> MX_Only:MXOnly-2.25U-Hotswap
- MX_LWIN1: renamed from MX_LWIN; value MX-NoLED -> MXOnly-1.25U-Hotswap; footprint (none) -> MX_Only:MXOnly-1.25U-Hotswap
- MX_M1: renamed from MX_M; footprint (none) -> MX_Only:MXOnly-1U-Hotswap
- MX_MENU1: renamed from MX_MENU; value MX-NoLED -> MXOnly-1.25U-Hotswap; footprint (none) -> MX_Only:MXOnly-1.25U-Hotswap
- MX_MINS1: renamed from MX_MINS; footprint (none) -> MX_Only:MXOnly-1U-FLIPPED
- MX_N1: renamed from MX_N; footprint (none) -> MX_Only:MXOnly-1U-FLIPPED
- MX_O1: renamed from MX_O; footprint (none) -> MX_Only:MXOnly-1U-FLIPPED
- MX_P1: renamed from MX_P; footprint (none) -> MX_Only:MXOnly-1U-FLIPPED
- MX_PAUS1: renamed from MX_PAUS; footprint (none) -> MX_Only:MXOnly-1U-FLIPPED
- MX_PGDN1: renamed from MX_PGDN; footprint (none) -> MX_Only:MXOnly-1U-FLIPPED
- MX_PGUP1: renamed from MX_PGUP; footprint (none) -> MX_Only:MXOnly-1U-FLIPPED
- MX_PSCR1: renamed from MX_PSCR; footprint (none) -> MX_Only:MXOnly-1U-FLIPPED
- MX_Q1: renamed from MX_Q; footprint (none) -> MX_Only:MXOnly-1U-FLIPPED
- MX_QUOT1: renamed from MX_QUOT; footprint (none) -> MX_Only:MXOnly-1U-FLIPPED
- MX_R1: renamed from MX_R; footprint (none) -> MX_Only:MXOnly-1U-FLIPPED
- MX_RALT1: renamed from MX_RALT; value MX-NoLED -> MXOnly-1.25U-Hotswap; footprint (none) -> MX_Only:MXOnly-1.25U-Hotswap
- MX_RBRC1: renamed from MX_RBRC; footprint (none) -> MX_Only:MXOnly-1U-Hotswap
- MX_RCTL1: renamed from MX_RCTL; value MX-NoLED -> MXOnly-1.25U-Hotswap; footprint (none) -> MX_Only:MXOnly-1.25U-Hotswap
- MX_RGHT1: renamed from MX_RGHT; footprint (none) -> MX_Only:MXOnly-1U-Hotswap
- MX_RSFT1: renamed from MX_RSFT; value MX-NoLED -> MXOnly-2.75U-Hotswap; footprint (none) -> MX_Only:MXOnly-2.25U-Hotswap
- MX_RWIN1: renamed from MX_RWIN; value MX-NoLED -> MXOnly-1.25U-Hotswap; footprint (none) -> MX_Only:MXOnly-1.25U-Hotswap
- MX_S1: renamed from MX_S; footprint (none) -> MX_Only:MXOnly-1U-Hotswap
- MX_SCLN1: renamed from MX_SCLN; footprint (none) -> MX_Only:MXOnly-1U-Hotswap
- MX_SLCK1: renamed from MX_SLCK; footprint (none) -> MX_Only:MXOnly-1U-Hotswap
- MX_SLSH1: renamed from MX_SLSH; footprint (none) -> MX_Only:MXOnly-1U-Hotswap
- MX_SPC1: renamed from MX_SPC; value MX-NoLED -> MXOnly-6.25U-Hotswap-ReversedStabilizers; footprint (none) -> MX_Only:MXOnly-6.25U-Hotswap-ReversedStabilizers
- MX_T1: renamed from MX_T; footprint (none) -> MX_Only:MXOnly-1U-Hotswap
- MX_TAB1: renamed from MX_TAB; value MX-NoLED -> MXOnly-1.5U-Hotswap; footprint (none) -> MX_Only:MXOnly-1.5U-Hotswap
- MX_U1: renamed from MX_U; footprint (none) -> MX_Only:MXOnly-1U-Hotswap
- MX_UP1: renamed from MX_UP; footprint (none) -> MX_Only:MXOnly-1U-Hotswap
- MX_V1: renamed from MX_V; footprint (none) -> MX_Only:MXOnly-1U-Hotswap
- MX_W1: renamed from MX_W; footprint (none) -> MX_Only:MXOnly-1U-Hotswap
- MX_X1: renamed from MX_X; footprint (none) -> MX_Only:MXOnly-1U-Hotswap
- MX_Y1: renamed from MX_Y; footprint (none) -> MX_Only:MXOnly-1U-Hotswap
- MX_Z1: renamed from MX_Z; footprint (none) -> MX_Only:MXOnly-1U-Hotswap
- R1, R2, R3, R4, R5, R6: renamed from R?; footprint (none) -> Resistor_SMD:R_0805_2012Metric
- SW1: renamed from SW?; footprint (none) -> random-keyboard-parts:SKQG-1155865
- USB1: renamed from USB?; footprint (none) -> Type-C:HRO-TYPE-C-31-M-12
- Y1: renamed from Y?; footprint (none) -> Crystal:Crystal_SMD_3225-4Pin_3.2x2.5mm
- gave numbers to parts that had none: 1
