File: Cognac Carl TKL+Macro Column Duplexed_USB_C.kicad_pcb (KiCad board)
At the start: 2 copper layers, 202 parts, among them SW1 SW_Push, U1 ATmega32U4-AU, Y1 16MHz

Commit message: Ran column traces, debating on whether to have columns on front or back of pcb
Parts:
- C1, C2, C3, C4, C5, C6, C7, F1, R1, R2, R3, R4, R5, R6, SW1, U1, Y1: moved to B.Cu
- moved U1 180.4 mm to (192.9, 63.5), turned to 270 degrees
- moved SW1 163.0 mm to (208.0, 53.2)
- moved R6 154.9 mm to (176.2, 52.4), turned to 90 degrees
- moved D50 150.9 mm to (390.5, 187.3), turned to 90 degrees
- moved D51 150.9 mm to (409.6, 187.3), turned to 90 degrees
- moved D67 150.9 mm to (69.8, 225.4), turned to 90 degrees
- moved D68 150.9 mm to (108.7, 225.4), turned to 90 degrees
- moved D69 150.9 mm to (139.7, 225.4), turned to 90 degrees
- moved D77 150.9 mm to (292.1, 225.4), turned to 90 degrees
- moved D85 150.9 mm to (218.3, 244.5), turned to 90 degrees
- moved R5 150.9 mm to (179.4, 52.4), turned to 90 degrees
- moved D35 150.1 mm to (69.8, 187.3), turned to 90 degrees
- moved D49 150.1 mm to (358.8, 187.3), turned to 90 degrees
- moved D52 150.1 mm to (428.6, 187.3), turned to 90 degrees
- moved D53 150.1 mm to (69.8, 206.4), turned to 90 degrees
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Routing:
- net COL5: track 0.00 -> 260.3 mm
- net COL1: track 0.00 -> 258.6 mm
- net COL7: track 0.00 -> 254.1 mm
- net COL3: track 0.00 -> 245.9 mm
- net COL6: track 0.00 -> 244.2 mm
- net COL0: track 0.00 -> 243.3 mm
- net COL4: track 0.00 -> 230.2 mm
- net COL2: track 0.00 -> 224.6 mm
- net COL8: track 0.00 -> 208.3 mm
Other:
- board outline added: 377.8 x 122.2 mm

Commit message: completed routing, removed hotswap, added esd protection
Parts:
- added C10: 0.1uF, Capacitor_SMD:C_0805_2012Metric, B.Cu at (366.4, 204.5)
- added C11: 0.1uF, Capacitor_SMD:C_0805_2012Metric, B.Cu at (363.7, 208.9)
- added C8: 0.1uF, Capacitor_SMD:C_0805_2012Metric, B.Cu at (383.4, 209.8)
- added U2: SRV05-4, Package_TO_SOT_SMD:SOT-23-6, B.Cu at (370.1, 196.0)
- D1, D10, D11, D12, D13, D14, D15, D16, D17, D18, D19, D2, D20, D21, D22, D23, D24, D25, D26, D27, D28, D29, D3, D30, D31, D32, D33, D34, D35, D36, D37, D38, D39, D4, D40, D41, D42, D43, D44, D45, D46, D47, D48, D49, D5, D50, D51, D52, D53, D54, D55, D56, D57, D58, D59, D6, D60, D61, D62, D63, D64, D65, D66, D67, D68, D69, D7, D70, D71, D72, D73, D74, D75, D76, D77, D78, D79, D8, D80, D81, D82, D83, D84, D85, D86, D87, D88, D89, D9, D90, D91, D92, USB1: moved to B.Cu
- MX1, MX12, MX13, MX14, MX15, MX17, MX18, MX19, MX2, MX20, MX21, MX23, MX24, MX25, MX26, MX27, MX28, MX29, MX3, MX30, MX31, MX32, MX33, MX34, MX35, MX36, MX37, MX38, MX39, MX4, MX40, MX41, MX42, MX44, MX45, MX46, MX47, MX48, MX49, MX5, MX50, MX51, MX52, MX53, MX54, MX55, MX56, MX57, MX58, MX59, MX6, MX60, MX61, MX63, MX65, MX66, MX67, MX68, MX7, MX70, MX71, MX72, MX74, MX80, MX81, MX82, MX83, MX84, MX85, MX86, MX87, MX88, MX89, MX90, MX91, MX92: footprint MX_Only:MXOnly-1U-Hotswap -> MX_Only:MXOnly-1U-NoLED
- MX10, MX77: footprint MX_Only:MXOnly-2.25U-Hotswap -> MX_Only:MXOnly-2.25U-NoLED
- MX11, MX16, MX22, MX64, MX69, MX73, MX79: footprint MX_Only:MXOnly-1.25U-Hotswap -> MX_Only:MXOnly-1.25U-NoLED
- MX43: footprint MX_Only:MXOnly-6.25U-Hotswap-ReversedStabilizers -> MX_Only:MXOnly-6.25U-ReversedStabilizers-NoLED
- MX62: value KC_SCOLON -> KC_SCOLON; footprint MX_Only:MXOnly-1U-Hotswap -> MX_Only:MXOnly-1U-NoLED
- MX75: footprint MX_Only:MXOnly-2U-Hotswap -> MX_Only:MXOnly-2U-NoLED
- MX76, MX8: footprint MX_Only:MXOnly-1.5U-Hotswap -> MX_Only:MXOnly-1.5U-NoLED
- MX78: footprint MX_Only:MXOnly-2.75U-Hotswap -> MX_Only:MXOnly-2.75U-NoLED
- MX9: footprint MX_Only:MXOnly-1.75U-Hotswap -> MX_Only:MXOnly-1.75U-NoLED
- moved C6 249.4 mm to (376.6, 221.1)
- moved SW1 244.0 mm to (398.5, 205.6)
- moved C4 240.8 mm to (376.6, 200.7), turned to 90 degrees
- moved C5 239.5 mm to (363.6, 217.9), turned to 90 degrees
- moved C1 238.4 mm to (387.1, 219.3)
- moved C2 238.4 mm to (387.1, 211.4)
- moved Y1 238.4 mm to (387.1, 215.4)
- moved R3 234.9 mm to (369.0, 202.1)
- moved R1 234.5 mm to (380.2, 207.3)
- moved R2 234.1 mm to (371.2, 202.1)
- moved R4 233.5 mm to (367.4, 222.6), turned to 90 degrees
- moved U1 233.4 mm to (372.1, 213.0)
- moved C3 233.3 mm to (374.4, 200.7)
- moved C7 225.2 mm to (366.6, 197.2), turned to 270 degrees
- moved R6 95.7 mm to (199.9, 145.1)
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Connections:
- U1 pad 10: Net-(U1-Pad10) -> COL3
- U1 pad 11: Net-(U1-Pad11) -> COL4
- U1 pad 18: Net-(U1-Pad18) -> COL8
- U1 pad 19: Net-(U1-Pad19) -> COL7
- U1 pad 20: Net-(U1-Pad20) -> COL6
- U1 pad 21: Net-(U1-Pad21) -> COL5
- U1 pad 25: Net-(U1-Pad25) -> COL1
- U1 pad 26: Net-(U1-Pad26) -> COL0
- U1 pad 27: Net-(U1-Pad27) -> ROW11
- U1 pad 28: Net-(U1-Pad28) -> ROW10
- U1 pad 29: Net-(U1-Pad29) -> ROW9
- U1 pad 30: Net-(U1-Pad30) -> ROW8
- U1 pad 31: Net-(U1-Pad31) -> ROW7
- U1 pad 32: Net-(U1-Pad32) -> ROW6
- U1 pad 36: Net-(U1-Pad36) -> ROW5
- U1 pad 37: Net-(U1-Pad37) -> ROW4
- U1 pad 38: Net-(U1-Pad38) -> ROW3
- U1 pad 39: Net-(U1-Pad39) -> ROW2
- U1 pad 40: Net-(U1-Pad40) -> ROW1
- U1 pad 41: Net-(U1-Pad41) -> ROW0
- U1 pad 9: Net-(U1-Pad9) -> COL2
Routing:
- net ROW1: track 0.00 -> 453.3 mm, vias 0 -> 4
- net GND: track 0.00 -> 431.4 mm, vias 0 -> 5
- net ROW3: track 0.00 -> 419.7 mm, vias 0 -> 2
- net ROW2: track 0.00 -> 411.7 mm, vias 0 -> 2
- net ROW4: track 0.00 -> 411.0 mm, vias 0 -> 2
- net ROW5: track 0.00 -> 392.7 mm, vias 0 -> 2
- net ROW11: track 0.00 -> 384.2 mm, vias 0 -> 2
- net ROW10: track 0.00 -> 381.5 mm, vias 0 -> 2
- net ROW0: track 0.00 -> 347.3 mm, vias 0 -> 2
- net ROW6: track 0.00 -> 343.7 mm, vias 0 -> 2
- net ROW9: track 0.00 -> 341.7 mm
- net ROW8: track 0.00 -> 340.1 mm
- net +5V: track 0.00 -> 339.7 mm, vias 0 -> 10
- net ROW7: track 0.00 -> 318.0 mm
- net COL0: track 243.3 -> 540.3 mm, vias 0 -> 5
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- added copper zone on B.Cu, net GND
- added copper zone on F.Cu, net GND
Other:
- board size 377.8 x 122.2 mm -> 376.2 x 123.8 mm
- net class Default: trace_width 0.25 -> 0.254
- net class Power added: clearance 0.2, trace_width 0.381, via_dia 0.8, via_drill 0.4

Commit message: replaced crytsal with a murata oscillator. tidied up routing, and added filled zones.
Parts:
- removed the C1 at (387.1, 219.3)
- removed the C2 at (387.1, 211.4)
- removed the C7 at (366.6, 197.2)
- removed the R5 at (196.8, 145.1)
- removed the R6 at (199.9, 145.1)
- added C8: 10uF, Capacitor_SMD:C_0805_2012Metric, B.Cu at (362.6, 205.1)
- added D93: LED, LED_SMD:LED_0805_2012Metric, B.Cu at (398.5, 206.4)
- added D94: LED, LED_SMD:LED_0805_2012Metric, B.Cu at (388.9, 206.4)
- added D95: LED, LED_SMD:LED_0805_2012Metric, B.Cu at (408.0, 206.4)
- added R2: 5.1k, Resistor_SMD:R_0805_2012Metric, B.Cu at (202.4, 145.6)
- added R3: 5.1k, Resistor_SMD:R_0805_2012Metric, B.Cu at (202.4, 143.3)
- added R7: R_Small, Resistor_SMD:R_0805_2012Metric, B.Cu at (398.5, 201.6)
- added R8: R_Small, Resistor_SMD:R_0805_2012Metric, B.Cu at (388.9, 201.6)
- added R9: R_Small, Resistor_SMD:R_0805_2012Metric, B.Cu at (408.0, 201.8)
- MX77: footprint MX_Only:MXOnly-2.25U-NoLED -> MX_Only:MXOnly-2.25U-ReversedStabilizers-NoLED
- Y1: footprint Crystal:Crystal_SMD_3225-4Pin_3.2x2.5mm -> Crystal:Resonator_SMD_muRata_CSTxExxV-3Pin_3.0x1.1mm
- moved F1 9.48 mm to (195.3, 149.8)
- moved SW1 7.14 mm to (398.5, 212.7), turned to 180 degrees
- moved C2 4.65 mm to (362.6, 207.1), turned to 180 degrees
- moved Y1 2.32 mm to (385.8, 213.5)
- moved R6 1.31 mm to (366.4, 221.7), turned to 0 degrees
- moved C1 1.18 mm to (362.6, 209.2), turned to 180 degrees
- moved C3 1.04 mm to (382.4, 210.2)
- moved C4 0.94 mm to (376.6, 199.7)
- moved C6 0.94 mm to (374.4, 199.7)
- renumbered C11 to C1, C10 to C2, C8 to C3, C3 to C6, C6 to C7, D17 to D1, D68 to D10, D82 to D11, D19 to D12, D37 to D13, D55 to D14, D69 to D15, D83 to D16, D2 to D17, D20 to D18, D38 to D19, D35 to D2, D56 to D20, D70 to D21, D84 to D22, D3 to D23, D21 to D24, D39 to D25, D57 to D26, D71 to D27, D4 to D28, D22 to D29, D53 to D3, D40 to D30, D58 to D31, D72 to D32, D5 to D33, D23 to D34, D41 to D35, D59 to D36, D73 to D37, D6 to D38, D24 to D39, D67 to D4, D42 to D40, D60 to D41, D74 to D42, D85 to D43, D7 to D44, D25 to D45, D43 to D46, D61 to D47, D75 to D48, D8 to D49, D81 to D5, D26 to D50, D44 to D51, D62 to D52, D76 to D53, D9 to D54, D27 to D55, D45 to D56, D63 to D57, D77 to D58, D10 to D59, D1 to D6, D28 to D60, D46 to D61, D64 to D62, D78 to D63, D86 to D64, D11 to D65, D29 to D66, D47 to D67, D65 to D68, D87 to D69, D18 to D7, D12 to D70, D30 to D71, D48 to D72, D88 to D73, D13 to D74, D31 to D75, D49 to D76, D66 to D77, D79 to D78, D89 to D79, D36 to D8, D14 to D80, D32 to D81, D50 to D82, D90 to D83, D15 to D84, D33 to D85, D51 to D86, D80 to D87, D91 to D88, D16 to D89, D54 to D9, D34 to D90, D52 to D91, R3 to R1, R2 to R4, R1 to R5, R4 to R6
Connections:
- net Net-(C1-Pad2) renamed XTAL1
- net Net-(C2-Pad2) renamed XTAL2
- U1 pad 18: COL8 -> Net-(U1-Pad18)
- U1 pad 19: COL7 -> COL8
- U1 pad 20: COL6 -> COL7
- U1 pad 21: COL5 -> COL6
- U1 pad 22: Net-(U1-Pad22) -> COL1
- U1 pad 25: COL1 -> ROW11
- U1 pad 26: COL0 -> ROW10
- U1 pad 27: ROW11 -> ROW9
- U1 pad 28: ROW10 -> ROW8
- U1 pad 29: ROW9 -> COL0
- U1 pad 30: ROW8 -> ROW7
- U1 pad 31: ROW7 -> ROW6
- U1 pad 32: ROW6 -> COL5
Routing:
- net GND: track 431.4 -> 317.9 mm, vias 5 -> 0
- net Net-(R9-Pad2): track 0.00 -> 62.0 mm, vias 0 -> 2
- net Net-(R7-Pad2): track 0.00 -> 29.6 mm
- net COL5: track 379.0 -> 351.8 mm, vias 5 -> 1
- net +5V: track 339.7 -> 360.8 mm, vias 10 -> 6
- net Net-(R8-Pad2): track 0.00 -> 15.6 mm
- net Net-(R5-Pad2): track 18.6 -> 32.0 mm
- net COL0: track 540.3 -> 532.9 mm, vias 5 -> 1
- net COL1: track 512.2 -> 519.3 mm, vias 7 -> 3
- net Net-(R2-Pad2): track 4.66 -> 11.6 mm, vias 0 -> 2
- net XTAL2: track 14.5 -> 8.00 mm
- net COL3: track 497.5 -> 492.8 mm
- net VCC: track 11.7 -> 16.4 mm
- net ROW0: track 347.3 -> 351.6 mm, vias 2 -> 4
- net XTAL1: track 12.9 -> 8.67 mm
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- added copper zone on B.Cu, net (none)
